File: Project/matrix.kicad_sch (KiCad schematic)
At the start: 92 parts, among them SW1 SW_Push_45deg, SW10 SW_Push_45deg, SW11 SW_Push_45deg, SW12 SW_Push_45deg, SW12(1.5)1 SW_Push_45deg, SW13 SW_Push_45deg, SW13(1.5)1 SW_Push_45deg, SW14 SW_Push_45deg, SW14(1.25)1 SW_Push_45deg, SW15 SW_Push_45deg, SW16 SW_Push_45deg, SW17 SW_Push_45deg, SW18 SW_Push_45deg, SW19 SW_Push_45deg, SW2 SW_Push_45deg, SW20 SW_Push_45deg, SW21 SW_Push_45deg, SW22 SW_Push_45deg, SW23 SW_Push_45deg, SW24 SW_Push_45deg, SW25 SW_Push_45deg, SW26 SW_Push_45deg, SW27 SW_Push_45deg, SW28 SW_Push_45deg, SW29 SW_Push_45deg, SW3 SW_Push_45deg, SW30 SW_Push_45deg, SW31 SW_Push_45deg, SW32 SW_Push_45deg, SW33 SW_Push_45deg, SW34 SW_Push_45deg, SW35 SW_Push_45deg, SW36 SW_Push_45deg, SW37(1.75)1 SW_Push_45deg, SW37(2.75)1 SW_Push_45deg, SW39 SW_Push_45deg, SW4 SW_Push_45deg, SW40 SW_Push_45deg, SW41 SW_Push_45deg, SW42 SW_Push_45deg, SW43 SW_Push_45deg, SW44 SW_Push_45deg, SW45 SW_Push_45deg, SW5 SW_Push_45deg, SW6 SW_Push_45deg, SW7 SW_Push_45deg, SW8 SW_Push_45deg, SW9 SW_Push_45deg

Commit message: changed footprints to ebastler
Parts:
- added S1, S3: MX_stab, PCM_marbastlib-mx:STAB_MX_P_3u, symbol PCM_marbastlib-mx:MX_stab
- added S2: MX_stab, PCM_marbastlib-mx:STAB_MX_P_7u, symbol PCM_marbastlib-mx:MX_stab
- added S4, S5: MX_stab, PCM_marbastlib-mx:STAB_MX_P_2.25u, symbol PCM_marbastlib-mx:MX_stab
- added S6: MX_stab, PCM_marbastlib-mx:STAB_MX_P_2.75u, symbol PCM_marbastlib-mx:MX_stab
- SW1, SW12(1.5)1, SW13(1.5)1, SW39, SW43: footprint MX_Only:MXOnly-1.5U-Hotswap -> PCM_marbastlib-mx:SW_MX_HS_1.5u
- SW10, SW11, SW12, SW13, SW15, SW16, SW17, SW18, SW19, SW2, SW20, SW21, SW22, SW23, SW24, SW27, SW28, SW29, SW3, SW30, SW31, SW32, SW33, SW34, SW35, SW36, SW4, SW40, SW42, SW5, SW6, SW7, SW8, SW9: footprint MX_Only:MXOnly-1U-Hotswap -> PCM_marbastlib-mx:SW_MX_HS_1u
- SW14, SW37(1.75)1: footprint MX_Only:MXOnly-1.75U-Hotswap -> PCM_marbastlib-mx:SW_MX_HS_1.75u
- SW14(1.25)1: footprint MX_Only:MXOnly-1.25U-Hotswap -> PCM_marbastlib-mx:SW_MX_HS_1.25u
- SW25, SW26: footprint MX_Only:MXOnly-2.25U-Hotswap -> PCM_marbastlib-mx:SW_MX_HS_1u
- SW37(2.75)1: footprint MX_Only:MXOnly-2.75U-Hotswap -> PCM_marbastlib-mx:SW_MX_HS_1u
- SW41: footprint MX_Only:MXOnly-7U-Hotswap-ReversedStabilizers -> PCM_marbastlib-mx:SW_MX_HS_1u
- SW44, SW45: footprint MX_Only:MXOnly-3U-Hotswap-ReversedStabilizers -> PCM_marbastlib-mx:SW_MX_HS_1u
Connections:
- net Col0: now also SW14(1.25)1.2; no longer SW14(1.25)1.1
- net Col11: now also SW12.2, SW37(1.75)1.2; no longer SW12.1, SW37(1.75)1.1
- net Col12: now also SW13(1.5)1.2; no longer SW13(1.5)1.1
- net at D43.2 (A), SW37(2.75)1.2: now also SW37(1.75)1.1; no longer SW37(1.75)1.2
- net at D41.2 (A), SW12(1.5)1.2: now also SW12.1; no longer SW12.2
- net at D3.2 (A), SW14.2: now also SW14(1.25)1.1; no longer SW14(1.25)1.2
- net at D44.2 (A), SW13.2: now also SW13(1.5)1.1; no longer SW13(1.5)1.2
Other:
- moved on the sheet: SW12, SW13(1.5)1, SW14(1.25)1, SW37(1.75)1
