File: Project/kira plate.kicad_pcb (KiCad board)
At the start: 2 copper layers, 266.7 x 85 mm, 1 part

Commit message: update
Parts:
- added REF**: MountingHole_2.2mm_M2, MountingHole:MountingHole_2.2mm_M2, F.Cu at (18.4, 107.1)
- added REF**: MountingHole_2.2mm_M2, MountingHole:MountingHole_2.2mm_M2, F.Cu at (276.9, 27.2)
- added REF**: MountingHole_2.2mm_M2, MountingHole:MountingHole_2.2mm_M2, F.Cu at (18.4, 27.2)
- added REF**: MountingHole_2.2mm_M2, MountingHole:MountingHole_2.2mm_M2, F.Cu at (276.9, 107.0)
- moved G*** 7.17 mm to (245.4, 93.0)
Other:
- outline, holes or cut-outs redrawn
